File: AFEIC.kicad_sch (KiCad schematic)
At the start: 37 parts, among them J4 CONN HEADER VERT 6POS 1.5MM, U1 TLE9012DQUXUMA1

Commit message: first layout
Connections:
- net BAT_GND is gone; now on net BATGND: C19.2
Changed lines of the file:
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@@
 		(in_pos_files yes)
 		(dnp no)
-		(fields_autoplaced yes)
 		(property "Reference" "#PWR013"
 			(at 151.13 205.74 0)
@@
 			)
 		)
-		(property "Value" "BAT_GND"
-			(at 151.13 204.47 0)
+		(property "Value" "BATGND"
+			(at 147.574 203.962 0)
 			(show_name no)
 			(do_not_autoplace no)
@@
 					(size 1.27 1.27)
 				)
+				(justify left)
 			)
 		)

Commit message: fixed minor layout changes
Connections:
- net IFL_H_Filt: no longer R22.1
- net IFL_L_Filt: no longer R23.1
- net IFH_H renamed IFH_P
- net IFH_H_Filt renamed IFH_Filt_P
- net IFH_L renamed IFH_N
- net IFH_L_Filt renamed IFH_Filt_N
- net IFL_H renamed IFL_P
- net IFL_L renamed IFL_N
- new net IFL_Filt_N: R23.1
- new net IFL_Filt_P: R22.1
Changed lines of the file:
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@@
 		)
 	)
-	(label "IFL_H_Filt"
+	(label "IFL_Filt_P"
 		(at 139.7 166.37 180)
 		(effects
@@
 		)
 	)
-	(label "IFH_L_Filt"
+	(label "IFH_Filt_N"
 		(at 72.39 91.44 180)
 		(effects
@@
 		)
 	)
-	(label "IFH_L_Filt"
+	(label "IFH_Filt_N"
 		(at 82.55 166.37 0)
 		(effects
@@
 		)
 	)
-	(label "IFL_L_Filt"
+	(label "IFL_Filt_N"
 		(at 139.7 189.23 180)
 		(effects
@@
 		)
 	)
-	(label "IFH_H_Filt"
+	(label "IFH_Filt_P"
 		(at 59.69 88.9 180)
 		(effects
@@
 		)
 	)
-	(label "IFH_H_Filt"
+	(label "IFH_Filt_P"
 		(at 82.55 191.77 0)
 		(effects
@@
 		)
 	)
-	(hierarchical_label "IFH_L"
+	(hierarchical_label "IFH_N"
 		(shape input)
 		(at 62.23 166.37 180)
@@
 		)
 	)
-	(hierarchical_label "IFL_L"
+	(hierarchical_label "IFL_N"
 		(shape input)
 		(at 161.29 189.23 0)
@@
 		)
 	)
-	(hierarchical_label "IFH_H"
+	(hierarchical_label "IFH_P"
 		(shape input)
 		(at 62.23 191.77 180)
@@
 		)
 	)
-	(hierarchical_label "IFL_H"
+	(hierarchical_label "IFL_P"
 		(shape input)
 		(at 161.29 166.37 0)

Commit message: minor layout changes
Parts:
- renumbered U1 to U8
Connections:
- net IFL_H_Filt is gone; now on net IFL_Filt_P: U8.24 (IFL_H)
- net IFL_L_Filt is gone; now on net IFL_Filt_N: U8.23 (IFL_L)
Changed lines of the file:
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@@
 		)
 	)
-	(label "IFL_H_Filt"
+	(label "IFL_Filt_P"
 		(at 158.75 72.39 0)
 		(effects
@@
 		)
 	)
-	(label "IFL_L_Filt"
+	(label "IFL_Filt_N"
 		(at 158.75 74.93 0)
 		(effects
@@
 		(dnp no)
 		(fields_autoplaced yes)
-		(property "Reference" "#PWR012"
+		(property "Reference" "#PWR12"
 			(at 151.13 182.88 0)
 			(hide yes)
@@
 			(project "bms-afe"
 				(path "/226a23e7-09bb-40bc-b53a-ec42a6b7cc90/0123e919-5cdb-453c-8cfd-f720a529864f"
-					(reference "#PWR012")
+					(reference "#PWR12")
 					(unit 1)
 				)
@@
 		(dnp no)
 		(fields_autoplaced yes)
-		(property "Reference" "#PWR029"
+		(property "Reference" "#PWR29"
 			(at 323.85 105.41 0)
 			(hide yes)
@@
 			(project "bms-afe"
 				(path "/226a23e7-09bb-40bc-b53a-ec42a6b7cc90/0123e919-5cdb-453c-8cfd-f720a529864f"
-					(reference "#PWR029")
+					(reference "#PWR29")
 					(unit 1)
 				)
@@
 		(dnp no)
 		(fields_autoplaced yes)
-		(property "Reference" "#PWR025"
+		(property "Reference" "#PWR25"
 			(at 271.78 105.41 0)
 			(hide yes)
@@
 			(project "bms-afe"
 				(path "/226a23e7-09bb-40bc-b53a-ec42a6b7cc90/0123e919-5cdb-453c-8cfd-f720a529864f"
-					(reference "#PWR025")
+					(reference "#PWR25")
 					(unit 1)
 				)
@@
 		(dnp no)
 		(fields_autoplaced yes)
-		(property "Reference" "#PWR024"
+		(property "Reference" "#PWR24"
 			(at 271.78 77.47 0)
 			(hide yes)
@@
 			(project "bms-afe"
 				(path "/226a23e7-09bb-40bc-b53a-ec42a6b7cc90/0123e919-5cdb-453c-8cfd-f720a529864f"
-					(reference "#PWR024")
+					(reference "#PWR24")
 					(unit 1)
 				)
@@
 		(in_pos_files yes)
 		(dnp no)
-		(property "Reference" "#PWR010"
+		(property "Reference" "#PWR10"
 			(at 90.17 114.3 0)
 			(hide yes)
@@
 			(project "bms-afe"
 				(path "/226a23e7-09bb-40bc-b53a-ec42a6b7cc90/0123e919-5cdb-453c-8cfd-f720a529864f"
-					(reference "#PWR010")
+					(reference "#PWR10")
 					(unit 1)
 				)
@@
 		(dnp no)
 		(fields_autoplaced yes)
-		(property "Reference" "#PWR022"
+		(property "Reference" "#PWR22"
 			(at 238.76 105.41 0)
 			(hide yes)
@@
 			(project "bms-afe"
 				(path "/226a23e7-09bb-40bc-b53a-ec42a6b7cc90/0123e919-5cdb-453c-8cfd-f720a529864f"
-					(reference "#PWR022")
+					(reference "#PWR22")
 					(unit 1)
 				)
@@
 		(dnp no)
 		(fields_autoplaced yes)
-		(property "Reference" "#PWR014"
+		(property "Reference" "#PWR14"
 			(at 156.21 105.41 0)
 			(hide yes)
@@
 			(project "bms-afe"
 				(path "/226a23e7-09bb-40bc-b53a-ec42a6b7cc90/0123e919-5cdb-453c-8cfd-f720a529864f"
-					(reference "#PWR014")
+					(reference "#PWR14")
 					(unit 1)
 				)
@@
 		(dnp no)
 		(fields_autoplaced yes)
-		(property "Reference" "U1"
+		(property "Reference" "U8"
 			(at 123.19 33.02 0)
 			(show_name no)
@@
 			(project "bms-afe"
 				(path "/226a23e7-09bb-40bc-b53a-ec42a6b7cc90/0123e919-5cdb-453c-8cfd-f720a529864f"
-					(reference "U1")
+					(reference "U8")
 					(unit 1)
 				)
@@
 		(dnp no)
 		(fields_autoplaced yes)
-		(property "Reference" "#PWR026"
+		(property "Reference" "#PWR26"
 			(at 283.21 105.41 0)
 			(hide yes)
@@
 			(project "bms-afe"
 				(path "/226a23e7-09bb-40bc-b53a-ec42a6b7cc90/0123e919-5cdb-453c-8cfd-f720a529864f"
-					(reference "#PWR026")
+					(reference "#PWR26")
 					(unit 1)
 				)
@@
 		(dnp no)
 		(fields_autoplaced yes)
-		(property "Reference" "#PWR027"
+		(property "Reference" "#PWR27"
 			(at 297.18 105.41 0)
 			(hide yes)
@@
 			(project "bms-afe"
 				(path "/226a23e7-09bb-40bc-b53a-ec42a6b7cc90/0123e919-5cdb-453c-8cfd-f720a529864f"
-					(reference "#PWR027")
+					(reference "#PWR27")
 					(unit 1)
 				)
@@
 		(dnp no)
 		(fields_autoplaced yes)
-		(property "Reference" "#PWR018"
+		(property "Reference" "#PWR18"
 			(at 187.96 105.41 0)
 			(hide yes)
@@
 			(project "bms-afe"
 				(path "/226a23e7-09bb-40bc-b53a-ec42a6b7cc90/0123e919-5cdb-453c-8cfd-f720a529864f"
-					(reference "#PWR018")
+					(reference "#PWR18")
 					(unit 1)
 				)
@@
 		(dnp no)
 		(fields_autoplaced yes)
-		(property "Reference" "#PWR09"
+		(property "Reference" "#PWR9"
 			(at 82.55 114.3 0)
 			(hide yes)
@@
 			(project "bms-afe"
 				(path "/226a23e7-09bb-40bc-b53a-ec42a6b7cc90/0123e919-5cdb-453c-8cfd-f720a529864f"
-					(reference "#PWR09")
+					(reference "#PWR9")
 					(unit 1)
 				)
@@
 		(dnp no)
 		(fields_autoplaced yes)
-		(property "Reference" "#PWR015"
+		(property "Reference" "#PWR15"
 			(at 165.1 105.41 0)
 			(hide yes)
@@
 			(project "bms-afe"
 				(path "/226a23e7-09bb-40bc-b53a-ec42a6b7cc90/0123e919-5cdb-453c-8cfd-f720a529864f"
-					(reference "#PWR015")
+					(reference "#PWR15")
 					(unit 1)
 				)
@@
 		(dnp no)
 		(fields_autoplaced yes)
-		(property "Reference" "#PWR011"
+		(property "Reference" "#PWR11"
 			(at 121.92 130.81 0)
 			(hide yes)
@@
 			(project "bms-afe"
 				(path "/226a23e7-09bb-40bc-b53a-ec42a6b7cc90/0123e919-5cdb-453c-8cfd-f720a529864f"
-					(reference "#PWR011")
+					(reference "#PWR11")
 					(unit 1)
 				)
@@
 		(dnp no)
 		(fields_autoplaced yes)
-		(property "Reference" "#PWR028"
+		(property "Reference" "#PWR28"
 			(at 308.61 105.41 0)
 			(hide yes)
@@
 			(project "bms-afe"
 				(path "/226a23e7-09bb-40bc-b53a-ec42a6b7cc90/0123e919-5cdb-453c-8cfd-f720a529864f"
-					(reference "#PWR028")
+					(reference "#PWR28")
 					(unit 1)
 				)
@@
 		(dnp no)
 		(fields_autoplaced yes)
-		(property "Reference" "#PWR016"
+		(property "Reference" "#PWR16"
 			(at 176.53 105.41 0)
 			(hide yes)
@@
 			(project "bms-afe"
 				(path "/226a23e7-09bb-40bc-b53a-ec42a6b7cc90/0123e919-5cdb-453c-8cfd-f720a529864f"
-					(reference "#PWR016")
+					(reference "#PWR16")
 					(unit 1)
 				)
@@
 		(dnp no)
 		(fields_autoplaced yes)
-		(property "Reference" "#PWR019"
+		(property "Reference" "#PWR19"
 			(at 201.93 105.41 0)
 			(hide yes)
@@
 			(project "bms-afe"
 				(path "/226a23e7-09bb-40bc-b53a-ec42a6b7cc90/0123e919-5cdb-453c-8cfd-f720a529864f"
-					(reference "#PWR019")
+					(reference "#PWR19")
 					(unit 1)
 				)
@@
 		(dnp no)
 		(fields_autoplaced yes)
-		(property "Reference" "#PWR07"
+		(property "Reference" "#PWR7"
 			(at 72.39 182.88 0)
 			(hide yes)
@@
 			(project "bms-afe"
 				(path "/226a23e7-09bb-40bc-b53a-ec42a6b7cc90/0123e919-5cdb-453c-8cfd-f720a529864f"
-					(reference "#PWR07")
+					(reference "#PWR7")
 					(unit 1)
 				)
@@
 		(dnp no)
 		(fields_autoplaced yes)
-		(property "Reference" "#PWR017"
+		(property "Reference" "#PWR17"
 			(at 181.61 72.39 0)
 			(hide yes)
@@
 			(project "bms-afe"
 				(path "/226a23e7-09bb-40bc-b53a-ec42a6b7cc90/0123e919-5cdb-453c-8cfd-f720a529864f"
-					(reference "#PWR017")
+					(reference "#PWR17")
 					(unit 1)
 				)
@@
 		(dnp no)
 		(fields_autoplaced yes)
-		(property "Reference" "#PWR030"
+		(property "Reference" "#PWR30"
 			(at 337.82 113.03 0)
 			(hide yes)
@@
 			(project "bms-afe"
 				(path "/226a23e7-09bb-40bc-b53a-ec42a6b7cc90/0123e919-5cdb-453c-8cfd-f720a529864f"
-					(reference "#PWR030")
+					(reference "#PWR30")
 					(unit 1)
 				)
@@
 		(in_pos_files yes)
 		(dnp no)
-		(property "Reference" "U1"
+		(property "Reference" "U8"
 			(at 350.266 61.214 0)
 			(show_name no)
@@
 			(project "bms-afe"
 				(path "/226a23e7-09bb-40bc-b53a-ec42a6b7cc90/0123e919-5cdb-453c-8cfd-f720a529864f"
-					(reference "U1")
+					(reference "U8")
 					(unit 2)
 				)
@@
 		(dnp no)
 		(fields_autoplaced yes)
-		(property "Reference" "#PWR020"
+		(property "Reference" "#PWR20"
 			(at 213.36 105.41 0)
 			(hide yes)
@@
 			(project "bms-afe"
 				(path "/226a23e7-09bb-40bc-b53a-ec42a6b7cc90/0123e919-5cdb-453c-8cfd-f720a529864f"
-					(reference "#PWR020")
+					(reference "#PWR20")
 					(unit 1)
 				)
@@
 		(dnp no)
 		(fields_autoplaced yes)
-		(property "Reference" "#PWR023"
+		(property "Reference" "#PWR23"
 			(at 241.3 182.88 0)
 			(hide yes)
@@
 			(project "bms-afe"
 				(path "/226a23e7-09bb-40bc-b53a-ec42a6b7cc90/0123e919-5cdb-453c-8cfd-f720a529864f"
-					(reference "#PWR023")
+					(reference "#PWR23")
 					(unit 1)
 				)
@@
 		(dnp no)
 		(fields_autoplaced yes)
-		(property "Reference" "#PWR021"
+		(property "Reference" "#PWR21"
 			(at 227.33 105.41 0)
 			(hide yes)
@@
 			(project "bms-afe"
 				(path "/226a23e7-09bb-40bc-b53a-ec42a6b7cc90/0123e919-5cdb-453c-8cfd-f720a529864f"
-					(reference "#PWR021")
+					(reference "#PWR21")
 					(unit 1)
 				)
@@
 		(in_pos_files yes)
 		(dnp no)
-		(property "Reference" "#PWR013"
+		(property "Reference" "#PWR13"
 			(at 151.13 205.74 0)
 			(hide yes)
@@
 			(project "bms-afe"
 				(path "/226a23e7-09bb-40bc-b53a-ec42a6b7cc90/0123e919-5cdb-453c-8cfd-f720a529864f"
-					(reference "#PWR013")
+					(reference "#PWR13")
 					(unit 1)
 				)
@@
 		(dnp no)
 		(fields_autoplaced yes)
-		(property "Reference" "#PWR08"
+		(property "Reference" "#PWR8"
 			(at 72.39 208.28 0)
 			(hide yes)
@@
 			(project "bms-afe"
 				(path "/226a23e7-09bb-40bc-b53a-ec42a6b7cc90/0123e919-5cdb-453c-8cfd-f720a529864f"
-					(reference "#PWR08")
+					(reference "#PWR8")
 					(unit 1)
 				)
