File: CellBalance.kicad_sch (KiCad schematic)
At the start: 9 parts

Commit message: initial component layout
Parts:
- renumbered C35 to C10, C12 to C9, R9 to R10, R45 to R6, R6 to R7, R7 to R8, R8 to R9
Other:
- note added: "= C_EMC (typical application) DNP for first balancing line"
- note removed: "= C_EMC (i used typical application)"

Commit message: minor layout changes
Parts:
- renumbered GSF1 to U1
Changed lines of the file:
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@@
 		(dnp no)
 		(fields_autoplaced yes)
-		(property "Reference" "#PWR05"
+		(property "Reference" "#PWR5"
 			(at 119.38 133.35 0)
 			(hide yes)
@@
 			(project "bms-afe"
 				(path "/226a23e7-09bb-40bc-b53a-ec42a6b7cc90/199aea63-5bfb-41be-ba55-0a021bc0a074"
-					(reference "#PWR031")
+					(reference "#PWR31")
 					(unit 1)
 				)
 				(path "/226a23e7-09bb-40bc-b53a-ec42a6b7cc90/2aa084bd-01e7-47e5-8f6d-30b4f325d7f4"
-					(reference "#PWR06")
+					(reference "#PWR6")
 					(unit 1)
 				)
 				(path "/226a23e7-09bb-40bc-b53a-ec42a6b7cc90/30f9ba51-47e3-4adb-895f-80ddd8089ec1"
-					(reference "#PWR033")
+					(reference "#PWR33")
 					(unit 1)
 				)
 				(path "/226a23e7-09bb-40bc-b53a-ec42a6b7cc90/9ef805d4-1601-4480-b9fd-3e26be539576"
-					(reference "#PWR034")
+					(reference "#PWR34")
 					(unit 1)
 				)
 				(path "/226a23e7-09bb-40bc-b53a-ec42a6b7cc90/a6f93463-0553-4e94-825f-86704d73fcd7"
-					(reference "#PWR05")
+					(reference "#PWR5")
 					(unit 1)
 				)
 				(path "/226a23e7-09bb-40bc-b53a-ec42a6b7cc90/cf97efbe-7ee9-4abe-8844-0d879c082204"
-					(reference "#PWR032")
+					(reference "#PWR32")
 					(unit 1)
 				)
@@
 		(dnp no)
 		(fields_autoplaced yes)
-		(property "Reference" "GSF1"
+		(property "Reference" "U1"
 			(at 132.08 76.1999 0)
 			(show_name no)
@@
 			(project "bms-afe"
 				(path "/226a23e7-09bb-40bc-b53a-ec42a6b7cc90/199aea63-5bfb-41be-ba55-0a021bc0a074"
-					(reference "GSF3")
+					(reference "U4")
 					(unit 1)
 				)
 				(path "/226a23e7-09bb-40bc-b53a-ec42a6b7cc90/2aa084bd-01e7-47e5-8f6d-30b4f325d7f4"
-					(reference "GSF2")
+					(reference "U3")
 					(unit 1)
 				)
 				(path "/226a23e7-09bb-40bc-b53a-ec42a6b7cc90/30f9ba51-47e3-4adb-895f-80ddd8089ec1"
-					(reference "GSF5")
+					(reference "U6")
 					(unit 1)
 				)
 				(path "/226a23e7-09bb-40bc-b53a-ec42a6b7cc90/9ef805d4-1601-4480-b9fd-3e26be539576"
-					(reference "GSF6")
+					(reference "U7")
 					(unit 1)
 				)
 				(path "/226a23e7-09bb-40bc-b53a-ec42a6b7cc90/a6f93463-0553-4e94-825f-86704d73fcd7"
-					(reference "GSF1")
+					(reference "U1")
 					(unit 1)
 				)
 				(path "/226a23e7-09bb-40bc-b53a-ec42a6b7cc90/cf97efbe-7ee9-4abe-8844-0d879c082204"
-					(reference "GSF4")
-					(unit 1)
-				)
+					(reference "U5")
+					(unit 1)
+				)
