File: bms-afe.kicad_sch (KiCad schematic)
At the start: 13 parts, among them J1 CONN HEADER VERT 7POS 2.5MM

Commit message: started layout
Parts:
- removed R1: RES 10 OHM 1% 1/10W 0603, Resistor_SMD:R_0603_1608Metric, symbol Device:R_Small_US
Connections:
- net CellBalance5/Battery_Pos is gone; now on net AFEIC/U12P: C11.2, C13.2, J1.7, R2.1
- net AFEIC/U12P: now also R3.1; no longer R3.2
- net VBLK: now also R3.2; no longer R3.1
Changed lines of the file:
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@@
+	)
+	(junction
+		(at 138.43 35.56)
+		(diameter 0)
+		(color 0 0 0 0)
 	)
 	(junction
@@
 		(color 0 0 0 0)
 	)
-	(junction
-		(at 138.43 31.75)
-		(diameter 0)
-		(color 0 0 0 0)
-	)
 	(wire
 		(pts
@@
 	(wire
 		(pts
-			(xy 173.99 31.75) (xy 173.99 58.42)
+			(xy 173.99 35.56) (xy 173.99 58.42)
 		)
 		(stroke
@@
 	(wire
 		(pts
-			(xy 115.57 31.75) (xy 115.57 43.18)
+			(xy 115.57 35.56) (xy 115.57 43.18)
 		)
 		(stroke
@@
 	(wire
 		(pts
-			(xy 138.43 24.13) (xy 138.43 31.75)
+			(xy 138.43 22.86) (xy 138.43 25.4)
 		)
 		(stroke
@@
 	(wire
 		(pts
-			(xy 173.99 31.75) (xy 149.86 31.75)
-		)
-		(stroke
-			(width 0)
-			(type default)
-		)
-	)
-	(wire
-		(pts
 			(xy 149.86 142.24) (xy 196.85 142.24)
 		)
@@
 	(wire
 		(pts
+			(xy 138.43 30.48) (xy 138.43 35.56)
+		)
+		(stroke
+			(width 0)
+			(type default)
+		)
+	)
+	(wire
+		(pts
 			(xy 115.57 55.88) (xy 121.92 55.88)
 		)
@@
 	(wire
 		(pts
-			(xy 127 31.75) (xy 115.57 31.75)
+			(xy 115.57 35.56) (xy 138.43 35.56)
 		)
 		(stroke
@@
 	(wire
 		(pts
-			(xy 138.43 31.75) (xy 144.78 31.75)
+			(xy 138.43 35.56) (xy 173.99 35.56)
 		)
 		(stroke
@@
 		(pts
 			(xy 81.28 113.03) (xy 86.36 113.03)
-		)
-		(stroke
-			(width 0)
-			(type default)
-		)
-	)
-	(wire
-		(pts
-			(xy 132.08 31.75) (xy 138.43 31.75)
 		)
 		(stroke
@@
 	)
 	(symbol
-		(lib_id "Device:R_Small_US")
-		(at 147.32 31.75 90)
-		(unit 1)
-		(body_style 1)
-		(exclude_from_sim no)
-		(in_bom yes)
-		(on_board yes)
-		(in_pos_files yes)
-		(dnp no)
-		(property "Reference" "R3"
-			(at 147.574 26.924 90)
-			(show_name no)
-			(do_not_autoplace no)
-			(effects
-				(font
-					(size 1.27 1.27)
-				)
-			)
-		)
-		(property "Value" "RES SMD 5.1 OHM 1% 1/8W 0603"
-			(at 159.512 28.956 90)
-			(show_name no)
-			(do_not_autoplace no)
-			(effects
-				(font
-					(size 1.27 1.27)
-				)
-			)
-		)
-		(property "Footprint" "Resistor_SMD:R_0603_1608Metric"
-			(at 147.32 31.75 0)
-			(hide yes)
-			(show_name no)
-			(do_not_autoplace no)
-			(effects
-				(font
-					(size 1.27 1.27)
-				)
-			)
-		)
-		(property "Datasheet" "https://www.digikey.ca/en/products/detail/vishay-dale/crcw06035r10fkea/1961617"
-			(at 147.32 31.75 0)
-			(hide yes)
-			(show_name no)
-			(do_not_autoplace no)
-			(effects
-				(font
-					(size 1.27 1.27)
-				)
-			)
-		)
-		(property "Description" "5.1 Ohms ±1% 0.125W, 1/8W Chip Resistor 0603 (1608 Metric) Automotive AEC-Q200 Thick Film"
-			(at 147.32 31.75 0)
-			(hide yes)
-			(show_name no)
-			(do_not_autoplace no)
-			(effects
-				(font
-					(size 1.27 1.27)
-				)
-			)
-		)
-		(property "LCSC" "C242492"
-			(at 147.32 31.75 0)
-			(hide yes)
-			(show_name no)
-			(do_not_autoplace no)
-			(effects
-				(font
-					(size 1.27 1.27)
-				)
-			)
-		)
-		(pin "2"
-		)
-		(pin "1"
-		)
-		(instances
-			(project "bms-afe"
-				(path "/226a23e7-09bb-40bc-b53a-ec42a6b7cc90"
-					(reference "R3")
-					(unit 1)
-				)
-			)
-		)
-	)
-	(symbol
 		(lib_id "symbols:B7B-XH-A_LF__SN_")
 		(at 73.66 113.03 180)
@@
 	(symbol
 		(lib_id "power:+3V3")
-		(at 138.43 24.13 0)
+		(at 138.43 22.86 0)
 		(unit 1)
 		(body_style 1)
@@
 		(fields_autoplaced yes)
 		(property "Reference" "#PWR04"
-			(at 138.43 27.94 0)
+			(at 138.43 26.67 0)
 			(hide yes)
 			(show_name no)
@@
 		)
 		(property "Value" "VBLK"
-			(at 138.43 19.05 0)
+			(at 138.43 17.78 0)
 			(show_name no)
 			(do_not_autoplace no)
@@
 		)
 		(property "Footprint" ""
-			(at 138.43 24.13 0)
+			(at 138.43 22.86 0)
 			(hide yes)
 			(show_name no)
@@
 		)
 		(property "Datasheet" ""
-			(at 138.43 24.13 0)
+			(at 138.43 22.86 0)
 			(hide yes)
 			(show_name no)
@@
 		)
 		(property "Description" "Power symbol creates a global label with name \"+3V3\""
-			(at 138.43 24.13 0)
+			(at 138.43 22.86 0)
 			(hide yes)
 			(show_name no)
@@
 	)
 	(symbol
+		(lib_id "Device:R_Small_US")
+		(at 138.43 27.94 180)
+		(unit 1)
+		(body_style 1)
+		(exclude_from_sim no)
+		(in_bom yes)
+		(on_board yes)
+		(in_pos_files yes)
+		(dnp no)
+		(property "Reference" "R3"
+			(at 142.24 27.432 0)
+			(show_name no)
+			(do_not_autoplace no)
+			(effects
+				(font
+					(size 1.27 1.27)
+				)
+			)
+		)
+		(property "Value" "RES SMD 5.1 OHM 1% 1/8W 0603"
+			(at 157.734 29.464 0)
+			(show_name no)
+			(do_not_autoplace no)
+			(effects
+				(font
+					(size 1.27 1.27)
+				)
+			)
+		)
+		(property "Footprint" "Resistor_SMD:R_0603_1608Metric"
+			(at 138.43 27.94 0)
+			(hide yes)
+			(show_name no)
+			(do_not_autoplace no)
+			(effects
+				(font
+					(size 1.27 1.27)
+				)
+			)
+		)
+		(property "Datasheet" "https://www.digikey.ca/en/products/detail/vishay-dale/crcw06035r10fkea/1961617"
+			(at 138.43 27.94 0)
+			(hide yes)
+			(show_name no)
+			(do_not_autoplace no)
+			(effects
+				(font
+					(size 1.27 1.27)
+				)
+			)
+		)
+		(property "Description" "5.1 Ohms ±1% 0.125W, 1/8W Chip Resistor 0603 (1608 Metric) Automotive AEC-Q200 Thick Film"
+			(at 138.43 27.94 0)
+			(hide yes)
+			(show_name no)
+			(do_not_autoplace no)
+			(effects
+				(font
+					(size 1.27 1.27)
+				)
+			)
+		)
+		(property "LCSC" "C242492"
+			(at 138.43 27.94 0)
+			(hide yes)
+			(show_name no)
+			(do_not_autoplace no)
+			(effects
+				(font
+					(size 1.27 1.27)
+				)
+			)
+		)
+		(pin "2"
+		)
+		(pin "1"
+		)
+		(instances
+			(project "bms-afe"
+				(path "/226a23e7-09bb-40bc-b53a-ec42a6b7cc90"
+					(reference "R3")
+					(unit 1)
+				)
+			)
+		)
+	)
+	(symbol
 		(lib_id "Device:C_Small")
 		(at 186.69 66.04 0)
@@
 					(unit 1)
 				)
-			)
-		)
-	)
-	(symbol
-		(lib_id "Device:R_Small_US")
-		(at 129.54 31.75 90)
-		(unit 1)
-		(body_style 1)
-		(exclude_from_sim no)
-		(in_bom yes)
-		(on_board yes)
-		(in_pos_files yes)
-		(dnp no)
-		(property "Reference" "R1"
-			(at 129.032 26.67 90)
-			(show_name no)
-			(do_not_autoplace no)
-			(effects
-				(font
-					(size 1.27 1.27)
-				)
-			)
-		)
-		(property "Value" "RES 10 OHM 1% 1/10W 0603"
-			(at 120.396 29.21 90)
-			(show_name no)
-			(do_not_autoplace no)
-			(effects
-				(font
-					(size 1.27 1.27)
-				)
-			)
-		)
-		(property "Footprint" "Resistor_SMD:R_0603_1608Metric"
-			(at 129.54 31.75 0)
-			(hide yes)
-			(show_name no)
-			(do_not_autoplace no)
-			(effects
-				(font
-					(size 1.27 1.27)
-				)
-			)
-		)
-		(property "Datasheet" "https://www.digikey.ca/en/products/detail/yageo/RC0603FR-0710RL/726879"
-			(at 129.54 31.75 0)
-			(hide yes)
-			(show_name no)
-			(do_not_autoplace no)
-			(effects
-				(font
-					(size 1.27 1.27)
-				)
-			)
-		)
-		(property "Description" "10 Ohms ±1% 0.1W, 1/10W Chip Resistor 0603 (1608 Metric) Moisture Resistant Thick Film"
-			(at 129.54 31.75 0)
-			(hide yes)
-			(show_name no)
-			(do_not_autoplace no)
-			(effects
-				(font
-					(size 1.27 1.27)
-				)
-			)
-		)
-		(pin "2"
-		)
-		(pin "1"
-		)
-		(instances
-			(project "bms-afe"
-				(path "/226a23e7-09bb-40bc-b53a-ec42a6b7cc90"
-					(reference "R1")
-					(unit 1)
-				)

Commit message: initial component layout
Parts:
- removed C60: CAP CER 0.33UF 25V X7R 0603, Capacitor_SMD:C_0603_1608Metric, symbol Device:C_Small
- added TP1, TP10, TP11, TP12, TP13, TP14, TP2, TP3, TP4, TP5, TP6, TP7, TP8, TP9: TestPoint, TestPoint:TestPoint_Pad_D1.0mm, symbol Connector:TestPoint
- renumbered C11 to C1, C13 to C2, C54 to C3, C55 to C4, C56 to C5, C57 to C6, C58 to C7, C59 to C8, R2 to R1, R3 to R2
Connections:
- net AFEIC/G0: now also TP14.1
- net AFEIC/G1: now also TP11.1
- net AFEIC/G2: now also TP9.1
- net AFEIC/G3: now also TP7.1
- net AFEIC/G4: now also TP5.1
- net AFEIC/G5: now also TP3.1
- net AFEIC/U0: now also TP13.1
- net AFEIC/U1: now also TP12.1
- net AFEIC/U12P: now also TP1.1
- net AFEIC/U2: now also TP10.1
- net AFEIC/U3: now also TP8.1
- net AFEIC/U4: now also TP6.1
- net AFEIC/U5: now also TP4.1
- net AFEIC/U6: now also TP2.1
Other:
- moved on the sheet: C1, C2, C3, C4, C5, C6, C7, C8, J1, R1, R2

Commit message: fixed minor layout changes
Other:
- sheet AFEIC ports: added IFH_N, IFH_P, IFL_N, IFL_P; removed IFH_H, IFH_L, IFL_H, IFL_L
- sheet BMSConn ports: added IFH_N, IFH_P, IFL_N, IFL_P; removed IFH_H, IFH_L, IFL_H, IFL_L
Changed lines of the file:
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@@
 			)
 		)
-		(pin "IFL_L" input
+		(pin "IFL_N" input
 			(at 229.87 66.04 0)
 			(effects
@@
 			)
 		)
-		(pin "IFL_H" input
+		(pin "IFL_P" input
 			(at 229.87 63.5 0)
 			(effects
@@
 			)
 		)
-		(pin "IFH_H" input
+		(pin "IFH_P" input
 			(at 229.87 72.39 0)
 			(effects
@@
 			)
 		)
-		(pin "IFH_L" input
+		(pin "IFH_N" input
 			(at 229.87 74.93 0)
 			(effects
@@
 			)
 		)
-		(pin "IFH_L" input
+		(pin "IFH_N" input
 			(at 241.3 74.93 180)
 			(effects
@@
 			)
 		)
-		(pin "IFH_H" input
+		(pin "IFH_P" input
 			(at 241.3 72.39 180)
 			(effects
@@
 			)
 		)
-		(pin "IFL_L" input
+		(pin "IFL_N" input
 			(at 241.3 66.04 180)
 			(effects
@@
 			)
 		)
-		(pin "IFL_H" input
+		(pin "IFL_P" input
 			(at 241.3 63.5 180)
 			(effects
