File: bms-afe.kicad_pcb (KiCad board)
At the start: 2 copper layers, 60.3 x 37.9 mm, 125 parts, among them J1 CONN HEADER VERT 7POS 2.5MM, J2 CONN HEADER VERT 2POS 1.5MM, J3 CONN HEADER VERT 2POS 1.5MM, J4 CONN HEADER VERT 6POS 1.5MM, T1 PULSE XFMR 15UH 1 OHM FOR PLC, U0 TestPoint, U1 MOSFET, P-CH, SINGLE, -4.1A, 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, U1 TestPoint, U2 TestPoint, U3 MOSFET, P-CH, SINGLE, -4.1A, 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, U3 TestPoint, U4 MOSFET, P-CH, SINGLE, -4.1A, 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, U4 TestPoint, U5 MOSFET, P-CH, SINGLE, -4.1A, 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, U5 TestPoint, U6 MOSFET, P-CH, SINGLE, -4.1A, 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, U6 TestPoint, U7 MOSFET, P-CH, SINGLE, -4.1A, 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, U8 TLE9012DQUXUMA1

Commit message: minor changes
Parts:
- moved J3 0.15 mm to (122.7, 103.5)
- moved J4 0.10 mm to (120.7, 96.4)
Routing:
- net /AFEIC/TMP2: track 20.3 -> 19.0 mm
Changed lines of the file:
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@@
 		(tags "test point SMD pad")
 		(property "Reference" "IFHN"
-			(at 0.5 -1.6 0)
+			(at 0.5 -1.5 0)
 			(layer "F.SilkS")
 			(effects
@@
 		(tags "capacitor")
 		(property "Reference" "C2"
-			(at -1.2 2.6125 180)
+			(at -1 3.7125 270)
 			(layer "F.SilkS")
 			(effects
@@
 	(footprint "footprints:CONN_B6B-ZR_JST"
 		(layer "F.Cu")
-		(at 120.7451 96.2977 180)
+		(at 120.7451 96.4 180)
 		(tags "B6B-ZR ")
 		(property "Reference" "J4"
@@
 	(footprint "footprints:CONN_B2B-ZR_02P_JST"
 		(layer "F.Cu")
-		(at 122.6 103.499999 -90)
+		(at 122.7477 103.4834 -90)
 		(tags "B2B-ZR ")
 		(property "Reference" "J3"
@@
 		(tags "resistor")
 		(property "Reference" "R4"
-			(at 0 -1.43 0)
+			(at 0 -1.299999 0)
 			(layer "F.SilkS")
 			(effects
@@
 		(tags "capacitor")
 		(property "Reference" "C1"
-			(at -1.2 3.4125 0)
+			(at -1 3.8125 90)
 			(layer "F.SilkS")
 			(effects
@@
 	)
 	(gr_line
-		(start 101.925001 92.7)
-		(end 79.2 92.7)
-		(stroke
-			(width 0.1)
-			(type default)
-		)
-		(layer "F.SilkS")
-	)
-	(gr_line
-		(start 101.925001 92.7)
-		(end 103.6 92.7)
-		(stroke
-			(width 0.1)
-			(type default)
-		)
-		(layer "F.SilkS")
-	)
-	(gr_line
 		(start 103.6 92.7)
 		(end 103.6 101.9)
@@
 	)
 	(gr_text "TEMP CONN"
-		(at 118.3 93.2 0)
+		(at 118.3 93.3 0)
 		(layer "F.SilkS")
 		(effects
@@
 	)
 	(segment
-		(start 99.875001 106.475001)
-		(end 99.075 106.475001)
-		(width 0.2)
-		(layer "F.Cu")
-		(net "Net-(U8A-TMP3)")
-	)
-	(segment
 		(start 101 107.6)
 		(end 99.875001 106.475001)
@@
 	)
 	(segment
-		(start 104.023836 107.617604)
+		(start 104.075 107.668768)
 		(end 104.006232 107.6)
 		(width 0.2)
@@
 		(net "Net-(U8A-TMP3)")
 	)
-	(via
-		(at 104.023836 107.617604)
-		(size 0.6)
-		(drill 0.3)
-		(layers "F.Cu" "B.Cu")
-		(net "Net-(U8A-TMP3)")
-	)
 	(segment
-		(start 104.2464 111.9464)
-		(end 105.025 111.9464)
+		(start 104.075 107.7)
+		(end 104.075 107.668768)
 		(width 0.2)
-		(layer "B.Cu")
+		(layer "F.Cu")
 		(net "Net-(U8A-TMP3)")
 	)
 	(segment
-		(start 104.2 107.833752)
-		(end 104.2 111.9)
+		(start 99.875001 106.475001)
+		(end 99.075 106.475001)
 		(width 0.2)
-		(layer "B.Cu")
+		(layer "F.Cu")
+		(net "Net-(U8A-TMP3)")
+	)
+	(via
+		(at 104.075 107.7)
+		(size 0.6)
+		(drill 0.3)
+		(layers "F.Cu" "B.Cu")
 		(net "Net-(U8A-TMP3)")
 	)
 	(segment
-		(start 104.2 111.9)
-		(end 104.2464 111.9464)
+		(start 104.075 107.7)
+		(end 104.075 111.775)
 		(width 0.2)
 		(layer "B.Cu")
@@
 	)
 	(segment
-		(start 104.023836 107.617604)
-		(end 104.023836 107.657588)
+		(start 104.2464 111.9464)
+		(end 105.025 111.9464)
 		(width 0.2)
 		(layer "B.Cu")
@@
 	)
 	(segment
-		(start 104.023836 107.657588)
-		(end 104.2 107.833752)
+		(start 104.075 111.775)
+		(end 104.2464 111.9464)
 		(width 0.2)
 		(layer "B.Cu")
@@
 	)
 	(segment
-		(start 108.473 107.625)
-		(end 108.473 106.627001)
+		(start 118.5 98.8)
+		(end 120.7451 96.5549)
 		(width 0.2)
 		(layer "B.Cu")
@@
 	)
 	(segment
-		(start 119.8 98.7)
-		(end 120.7451 97.7549)
+		(start 109.075 107.625)
+		(end 117.9 98.8)
 		(width 0.2)
 		(layer "B.Cu")
@@
 	)
 	(segment
-		(start 120.7451 97.7549)
+		(start 120.7451 96.5549)
 		(end 120.7451 96.2977)
 		(width 0.2)
@@
 	)
 	(segment
-		(start 116.400001 98.7)
-		(end 119.8 98.7)
+		(start 117.9 98.8)
+		(end 118.5 98.8)
 		(width 0.2)
 		(layer "B.Cu")
@@
 	)
 	(segment
-		(start 108.473 106.627001)
-		(end 116.400001 98.7)
+		(start 108.473 107.625)
+		(end 109.075 107.625)
 		(width 0.2)
 		(layer "B.Cu")
@@
 	)
 	(segment
-		(start 103.125 107.9464)
-		(end 103.125 109.977)
+		(start 103.225 107.8464)
+		(end 103.225 107.175)
 		(width 0.2)
 		(layer "B.Cu")
@@
 	)
 	(segment
-		(start 103.225 107.175)
-		(end 106.625 103.775)
+		(start 103.125 107.9464)
+		(end 103.125 109.977)
 		(width 0.2)
 		(layer "B.Cu")
@@
 	)
 	(segment
-		(start 117.745101 97.354899)
+		(start 117.745101 97.154899)
 		(end 117.745101 96.2977)
 		(width 0.2)
@@
 	)
 	(segment
-		(start 116.234316 98.3)
-		(end 116.8 98.3)
-		(width 0.2)
-		(layer "B.Cu")
-		(net "/AFEIC/TMP0")
-	)
-	(segment
-		(start 103.225 107.8464)
-		(end 103.225 107.175)
-		(width 0.2)
-		(layer "B.Cu")
-		(net "/AFEIC/TMP0")
-	)
-	(segment
-		(start 103.125 107.9464)
-		(end 103.225 107.8464)
+		(start 103.225 107.175)
+		(end 106.625 103.775)
 		(width 0.2)
 		(layer "B.Cu")
@@
 	(segment
 		(start 106.625 103.775)
-		(end 110.759315 103.775)
+		(end 111.125 103.775)
 		(width 0.2)
 		(layer "B.Cu")
@@
 	)
 	(segment
-		(start 116.8 98.3)
-		(end 117.745101 97.354899)
+		(start 103.125 107.9464)
+		(end 103.225 107.8464)
 		(width 0.2)
 		(layer "B.Cu")
@@
 	)
 	(segment
-		(start 110.759315 103.775)
-		(end 116.234316 98.3)
+		(start 111.125 103.775)
+		(end 117.745101 97.154899)
 		(width 0.2)
 		(layer "B.Cu")

Commit message: added logo
Parts:
- added G***: LOGO, footprints:electriumlogo12, F.Cu at (72.1, 97.3)
- added G***: LOGO, footprints:dog, B.Cu at (71.5, 124.4)
